File: hardware/PCB/STIC/STIC.sch (KiCad schematic (older format))
At the start: 12 parts, among them J1 DIP-JST-2P-2.0, J2 Button connector, J3 Laser A, J4 Laser B, Q1 Q_PMOS_GSD, U1 XIAO_BLE, U2 RM3100_Breakout, U3 MDOB048064AV

Commit message: More work on PCB and schematic
Fat boy made and working!
Connections:
- net BUTTON: now also U1.4 (P0.29_A3_D3); no longer U1.3 (P0.28_A2_D2)
- net LED2_R: now also U1.5 (P0.04_A4_D4_SDA); no longer U1.4 (P0.29_A3_D3)
- net PERIPH_EN: now also U1.2 (P0.03_A1_D1); no longer U1.7 (P1.11_D6_TX)
- net SCL: now also U1.7 (P1.11_D6_TX); no longer U1.5 (P0.04_A4_D4_SDA)
- net at LS1.1: now also U1.3 (P0.28_A2_D2); no longer U1.2 (P0.03_A1_D1)
Changed lines of the file:
@@
 	5500 3400 5900 3400
-Wire Wire Line
-	3850 2800 3500 2800
 Wire Wire Line
 	3850 2950 3500 2950
@@
 	-1   0    0    1
 $EndComp
-Wire Wire Line
-	3300 2650 3300 2350
-Wire Wire Line
-	3300 2350 3100 2350
-Wire Wire Line
-	3300 2650 3850 2650
 $Comp
 L Device:Q_PMOS_GSD Q1
@@
 	0    1    1    0
 $EndComp
-Text Label 3500 3400 2    50   ~ 0
+Text Label 3500 2650 2    50   ~ 0
 PERIPH_EN
-Text Label 3500 2800 2    50   ~ 0
+Text Label 3500 2950 2    50   ~ 0
 BUTTON
 Text Label 5900 3100 0    50   ~ 0
@@
 Text Label 8550 2250 2    50   ~ 0
 BUTTON
-Text Label 3500 2950 2    50   ~ 0
+Text Label 3500 3100 2    50   ~ 0
 LED2_R
 Text Label 5900 3400 0    50   ~ 0
@@
 Text Label 3500 3250 2    50   ~ 0
 SDA
-Text Label 3500 3100 2    50   ~ 0
+Text Label 3500 3400 2    50   ~ 0
 SCL
 Wire Wire Line
@@
 	1    0    0    -1
 $EndComp
+Wire Wire Line
+	3850 2650 3500 2650
+Wire Wire Line
+	3850 2800 3650 2800
+Wire Wire Line
+	3650 2800 3650 2350
+Wire Wire Line
+	3100 2350 3650 2350
 $EndSCHEMATC
