File: hardware/PCB/STIC/STIC.kicad_pcb (KiCad board)
At the start: 2 copper layers, 12 parts, among them J1 DIP-JST-2P-2.0, J2 Button connector, J3 Laser A, J4 Laser B, Q1 Q_PMOS_GSD, U1 XIAO_BLE, U2 RM3100_Breakout, U3 MDOB048064AV

Commit message: More work on PCB and schematic
Fat boy made and working!
Parts:
- moved U3 20.9 mm to (106.7, 105.3)
Connections:
- U1 pad 2: Net-(LS1-Pad1) -> /PERIPH_EN
- U1 pad 3: /BUTTON -> Net-(LS1-Pad1)
- U1 pad 4: /LED2_R -> /BUTTON
- U1 pad 5: /SCL -> /LED2_R
- U1 pad 7: /PERIPH_EN -> /SCL
Routing:
- net +3V3: track 80.7 -> 111.0 mm
- net GND: track 13.3 -> 34.9 mm
- net +3.3VA: track 43.0 -> 22.4 mm
- net /SCL: track 73.8 -> 55.9 mm
- net /PERIPH_EN: track 23.2 -> 35.2 mm
- net /LED2_R: track 74.9 -> 65.5 mm
- net +BATT: track 60.2 -> 68.5 mm
- net Net-(J4-Pad1): track 0.00 -> 7.80 mm
- net Net-(J3-Pad6): track 0.00 -> 7.70 mm
- net /Rx: track 80.8 -> 88.5 mm
- net Net-(J4-Pad4): track 0.00 -> 7.67 mm
- net Net-(J4-Pad3): track 0.00 -> 7.60 mm
- net Net-(J3-Pad2): track 0.00 -> 7.60 mm
- net Net-(J3-Pad3): track 0.00 -> 7.50 mm
- net Net-(J4-Pad7): track 0.00 -> 7.40 mm
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Other:
- board outline added: 38.3 x 80.9 mm

Commit message: Update main PCB design
Other:
- board size 38.3 x 80.9 mm -> 38 x 80 mm
Changed lines of the file:
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@@
   (general
     (thickness 1.6)
-    (drawings 4)
+    (drawings 9)
     (tracks 222)
     (zones 0)
@@
   )
   (setup
-    (last_trace_width 1)
+    (last_trace_width 0.25)
     (user_trace_width 0.5)
     (user_trace_width 1)
@@
     (pad 2 thru_hole circle (at 10 0 90) (size 2 2) (drill 1) (layers *.Cu *.Mask)
       (net 10 "Net-(LS1-Pad2)"))
-    (model ${KISYS3DMOD}/Buzzer_Beeper.3dshapes/Buzzer_D14mm_H7mm_P10mm.wrl
+    (model ${KISYS3DMOD}/Buzzer_Beeper.3dshapes/Buzzer_15x7.5RM7.6.wrl
       (at (xyz 0 0 0))
       (scale (xyz 1 1 1))
@@
     )
   )
-  (gr_line (start 123.15 139.35) (end 84.85 139.35) (layer Edge.Cuts) (width 0.05))
-  (gr_line (start 84.85 139.35) (end 84.85 58.45) (layer Edge.Cuts) (width 0.05))
-  (gr_line (start 123.05 58.45) (end 123.15 139.35) (layer Edge.Cuts) (width 0.05))
-  (gr_line (start 84.85 58.45) (end 123.05 58.45) (layer Edge.Cuts) (width 0.05))
+  (gr_circle (center 104.95 115.34) (end 105.68 114.02) (layer Edge.Cuts) (width 0.05))
+  (gr_line (start 84.75 136.75) (end 84.75 60.75) (layer Edge.Cuts) (width 0.05))
+  (gr_line (start 86.75 138.75) (end 84.75 136.75) (layer Edge.Cuts) (width 0.05))
+  (gr_line (start 120.75 138.75) (end 86.75 138.75) (layer Edge.Cuts) (width 0.05))
+  (gr_line (start 122.75 136.75) (end 120.75 138.75) (layer Edge.Cuts) (width 0.05))
+  (gr_line (start 122.75 60.75) (end 122.75 136.75) (layer Edge.Cuts) (width 0.05))
+  (gr_line (start 120.75 58.75) (end 122.75 60.75) (layer Edge.Cuts) (width 0.05))
+  (gr_line (start 86.75 58.75) (end 120.75 58.75) (layer Edge.Cuts) (width 0.05))
+  (gr_line (start 84.75 60.75) (end 86.75 58.75) (layer Edge.Cuts) (width 0.05))
   (via (at 104.95 115.35) (size 6) (drill 3) (layers F.Cu B.Cu) (net 0))
   (segment (start 93.45 136.05) (end 93.45 140.15) (width 1.25) (layer F.Cu) (net 1))
-  (segment (start 108.85 136.15) (end 108.85 139.95) (width 1.25) (layer F.Cu) (net 2))
-  (segment (start 107.35 136.95) (end 107.35 139.85) (width 1.25) (layer F.Cu) (net 3))
-  (segment (start 96.45 136.05) (end 96.45 138.235) (width 1.25) (layer F.Cu) (net 4))
-  (segment (start 96.45 138.235) (end 96.45 139.95) (width 1.25) (layer F.Cu) (net 4))
-  (segment (start 105.85 136.15) (end 105.85 139.95) (width 1.25) (layer F.Cu) (net 25))
-  (segment (start 110.35 136.15) (end 110.35 139.85) (width 1.25) (layer F.Cu) (net 26))
-  (segment (start 111.85 136.05) (end 111.85 139.85) (width 1.25) (layer F.Cu) (net 27))
-  (segment (start 113.35 136.05) (end 113.35 139.75) (width 1.25) (layer F.Cu) (net 28))
-  (segment (start 94.95 136.65) (end 94.95 140.05) (width 1.25) (layer F.Cu) (net 29))
-  (segment (start 97.95 136.45) (end 97.95 139.95) (width 1.25) (layer F.Cu) (net 30))
-  (segment (start 99.40001 136.19999) (end 99.40001 139.95) (width 1.25) (layer F.Cu) (net 31))
-  (segment (start 100.95 136.05) (end 100.95 139.85) (width 1.25) (layer F.Cu) (net 32))
-  (segment (start 102.45 136.55) (end 102.45 139.85) (width 1.25) (layer F.Cu) (net 33))
-  (segment (start 103.95 136.05) (end 103.95 139.95) (width 1.25) (layer F.Cu) (net 34))
   (segment (start 110.79768 65.95218) (end 113.84782 65.95218) (width 1) (layer F.Cu) (net 1))
   (via (at 113.84782 65.95218) (size 2) (drill 1) (layers F.Cu B.Cu) (net 1))
@@
   (segment (start 102.65 96.85) (end 105.95 96.85) (width 1) (layer F.Cu) (net 1))
   (segment (start 99.07 100.43) (end 102.65 96.85) (width 1) (layer F.Cu) (net 1))
-  (via (at 98.85 71.85) (size 3) (drill 2) (layers F.Cu B.Cu) (net 23))
+  (segment (start 108.85 136.15) (end 108.85 139.95) (width 1.25) (layer F.Cu) (net 2))
   (segment (start 109.15 134.45) (end 108.85 134.75) (width 0.5) (layer F.Cu) (net 2))
   (segment (start 113.35 132.95) (end 111.85 134.45) (width 0.5) (layer F.Cu) (net 2))
@@
   (segment (start 108.85 136.05) (end 108.85 136.15) (width 1.25) (layer B.Cu) (net 2))
   (segment (start 108.85 136.15) (end 108.85 139.95) (width 1.25) (layer B.Cu) (net 2))
+  (segment (start 107.35 136.95) (end 107.35 139.85) (width 1.25) (layer F.Cu) (net 3))
   (segment (start 107.35 134.66499) (end 107.35 136.05) (width 0.5) (layer F.Cu) (net 3))
   (segment (start 107.35 134.25) (end 107.35 134.66499) (width 0.5) (layer F.Cu) (net 3))
@@
   (segment (start 107.35 136.05) (end 107.35 136.95) (width 1.25) (layer B.Cu) (net 3))
   (segment (start 107.35 136.95) (end 107.35 139.85) (width 1.25) (layer B.Cu) (net 3))
+  (segment (start 96.45 136.05) (end 96.45 138.235) (width 1.25) (layer F.Cu) (net 4))
+  (segment (start 96.45 138.235) (end 96.45 139.95) (width 1.25) (layer F.Cu) (net 4))
   (segment (start 109.25 100.75) (end 109.25 100.75) (width 0.25) (layer F.Cu) (net 4))
   (via (at 109.35 94.55) (size 2) (drill 1) (layers F.Cu B.Cu) (net 4))
@@
   (segment (start 103.25 92.85) (end 102.45 92.05) (width 0.5) (layer F.Cu) (net 19))
   (segment (start 105.95 92.85) (end 103.25 92.85) (width 0.5) (layer F.Cu) (net 19))
+  (via (at 98.85 71.85) (size 3) (drill 2) (layers F.Cu B.Cu) (net 23))
   (segment (start 98.85 80.95) (end 98.85 71.85) (width 2) (layer B.Cu) (net 23))
   (segment (start 101.55 83.55) (end 101.45 83.55) (width 2) (layer B.Cu) (net 23))
@@
   (segment (start 111.44218 68.45) (end 111.4 68.49218) (width 2) (layer F.Cu) (net 24))
   (segment (start 114.15 68.45) (end 111.44218 68.45) (width 2) (layer F.Cu) (net 24))
+  (segment (start 105.85 136.15) (end 105.85 139.95) (width 1.25) (layer F.Cu) (net 25))
   (segment (start 105.85 136.05) (end 105.85 136.15) (width 1.25) (layer B.Cu) (net 25))
   (segment (start 105.85 136.15) (end 105.85 139.95) (width 1.25) (layer B.Cu) (net 25))
+  (segment (start 110.35 136.15) (end 110.35 139.85) (width 1.25) (layer F.Cu) (net 26))
   (segment (start 110.35 136.05) (end 110.35 136.15) (width 1.25) (layer B.Cu) (net 26))
   (segment (start 110.35 136.15) (end 110.35 139.85) (width 1.25) (layer B.Cu) (net 26))
+  (segment (start 111.85 136.05) (end 111.85 139.85) (width 1.25) (layer F.Cu) (net 27))
   (segment (start 111.85 136.05) (end 111.85 139.85) (width 1.25) (layer B.Cu) (net 27))
+  (segment (start 113.35 136.05) (end 113.35 139.75) (width 1.25) (layer F.Cu) (net 28))
   (segment (start 113.35 136.05) (end 113.35 139.75) (width 1.25) (layer B.Cu) (net 28))
+  (segment (start 94.95 136.65) (end 94.95 140.05) (width 1.25) (layer F.Cu) (net 29))
   (segment (start 94.95 136.05) (end 94.95 136.65) (width 1.25) (layer B.Cu) (net 29))
   (segment (start 94.95 136.65) (end 94.95 140.05) (width 1.25) (layer B.Cu) (net 29))
+  (segment (start 97.95 136.45) (end 97.95 139.95) (width 1.25) (layer F.Cu) (net 30))
   (segment (start 97.95 136.05) (end 97.95 136.45) (width 1.25) (layer B.Cu) (net 30))
   (segment (start 97.95 136.45) (end 97.95 139.95) (width 1.25) (layer B.Cu) (net 30))
+  (segment (start 99.40001 136.19999) (end 99.40001 139.95) (width 1.25) (layer F.Cu) (net 31))
   (segment (start 99.45 136.15) (end 99.40001 136.19999) (width 1.25) (layer B.Cu) (net 31))
   (segment (start 99.45 136.05) (end 99.45 136.15) (width 1.25) (layer B.Cu) (net 31))
   (segment (start 99.40001 136.19999) (end 99.40001 139.95) (width 1.25) (layer B.Cu) (net 31))
+  (segment (start 100.95 136.05) (end 100.95 139.85) (width 1.25) (layer F.Cu) (net 32))
   (segment (start 100.95 136.05) (end 100.95 139.85) (width 1.25) (layer B.Cu) (net 32))
+  (segment (start 102.45 136.55) (end 102.45 139.85) (width 1.25) (layer F.Cu) (net 33))
   (segment (start 102.45 136.05) (end 102.45 136.55) (width 1.25) (layer B.Cu) (net 33))
   (segment (start 102.45 136.55) (end 102.45 139.85) (width 1.25) (layer B.Cu) (net 33))
+  (segment (start 103.95 136.05) (end 103.95 139.95) (width 1.25) (layer F.Cu) (net 34))
   (segment (start 103.95 136.05) (end 103.95 139.95) (width 1.25) (layer B.Cu) (net 34))
-  (zone (net 1) (net_name GND) (layer B.Cu) (hatch edge 0.508)
+  (zone (net 0) (net_name "") (layer B.Cu) (hatch edge 0.508)
     (connect_pads (clearance 0.508))
     (min_thickness 0.254)
-    (fill yes (arc_segments 32) (thermal_gap 0.508) (thermal_bridge_width 0.508))
+    (keepout (tracks not_allowed) (vias not_allowed) (copperpour not_allowed))
+    (fill (arc_segments 32) (thermal_gap 0.508) (thermal_bridge_width 0.508))
     (polygon
       (pts
-        (xy 122.75 138.75) (xy 85.25 138.75) (xy 85.25 58.75) (xy 122.75 58.75)
+        (xy 104.05 101.85) (xy 91.55 101.85) (xy 91.55 85.95) (xy 104.05 85.95)
       )
     )
   )
-  (zone (net 0) (net_name "") (layer B.Cu) (hatch edge 0.508)
+  (zone (net 1) (net_name GND) (layer B.Cu) (hatch edge 0.508)
     (connect_pads (clearance 0.508))
     (min_thickness 0.254)
-    (keepout (tracks not_allowed) (vias not_allowed) (copperpour not_allowed))
-    (fill (arc_segments 32) (thermal_gap 0.508) (thermal_bridge_width 0.508))
+    (fill yes (arc_segments 32) (thermal_gap 0.508) (thermal_bridge_width 0.508))
     (polygon
       (pts
-        (xy 104.05 101.85) (xy 91.55 101.85) (xy 91.55 85.95) (xy 104.05 85.95)
+        (xy 122.75 138.75) (xy 85.25 138.75) (xy 85.25 58.75) (xy 122.75 58.75)
       )
     )
