File: hardware/PCB/STIC.kicad_pcb (KiCad board)
At the start: 2 copper layers, 38 x 80 mm, 15 parts, among them J1 22-03-5035, J2 53047-0510, J3 53047-0310, U1 XIAO_BLE, U2 RM3100_Breakout, U3 OLED1_3_GND1

Commit message: Various PCB work
Add laser and battery to schematic (but not board, obvs)
Add second battery connector to allow JST-PH2 connectors
Add helpful silkscreen to board
Parts:
- added J5: Conn_01x02, Connector_JST:JST_PH_B2B-PH-K_1x02_P2.00mm_Vertical, F.Cu at (105.0, 123.3)
Routing:
- net +BATT: track 74.7 -> 76.6 mm
Other:
- board text added: "+"
- board text added: "-"
- board text added: "3.3V"
- board text added: "BATT"
- board text added: "Buttons"
- board text added: "Buzzer"
- board text added: "GND"
- board text added: "Laser"
- board text added: "RM3100"
- board text added: "SAP 6.2"
- board text added: "SCL"
- board text added: "SDA"
- board text removed: "SAP 6.1"
