File: hardware/PCB/STIC.kicad_sch (KiCad schematic)
At the start: 27 parts, among them J1 22-03-5035, J2 53047-0510, J3 53047-0310, J4 3 way molex cable, J5 Conn_01x02, J6 5 way molex cable, U1 XIAO_BLE, U2 RM3100_Breakout, U3 OLED1_3_GND1, U4 XIAO_RM3100_Breakout

Commit message: Working on 6A
Parts:
- removed C_1, C_2: 1.0uF, Capacitor_THT:C_Disc_D5.0mm_W2.5mm_P2.50mm, symbol Device:C
- removed C_3: 4.7uF, Capacitor_THT:C_Disc_D5.0mm_W2.5mm_P2.50mm, symbol Device:C
- removed R_1, R_2, R_3: 2k, Resistor_THT:R_Axial_DIN0204_L3.6mm_D1.6mm_P5.08mm_Horizontal, symbol Device:R
- removed U1: XIAO_BLE, XIAO:Seeeduino_XIAO-MOUDLE14P-2.54-21X17.8MM, symbol STIC-rescue:XIAO_BLE-XIAO
- added C1, C2: 100nf, Capacitor_SMD:C_0603_1608Metric, symbol Device:C
- added C3: 4.7uF, Capacitor_SMD:C_0603_1608Metric, symbol Device:C
- added U1: ASM330LHHTR, Package_LGA:LGA-14_3x2.5mm_P0.5mm_LayoutBorder3x4y, symbol ASM330LHHTR:ASM330LHHTR
- added U2: XIAO-ESP32-S3-SMD, Seeeduino XIAO KICAD:XIAO-ESP32-S3-SMD_PAD, symbol Seeed_Studio_XIAO_Series_kicad8:XIAO-ESP32-S3-SMD
- C4: renamed from C1; Seeed Part Number (none) -> 302011726
- C5: renamed from C2; Seeed Part Number (none) -> 302011726
- C6: renamed from C3; Seeed Part Number (none) -> 302012206
- CHARGER1: Seeed Part Number (none) -> XC6802A42XMR-G
- J3: renamed from J2; value 53047-0510 -> 53398-0571; footprint Connector_Molex:Molex_PicoBlade_53047-0510_1x05_P1.25mm_Vertical -> Connector_Molex:Molex_PicoBlade_53398-0571_1x05-1MP_P1.25mm_Vertical; Allied_Number 70266929 -> (none); Farnell Part Number 9732861 -> (none); Manufacturer_Part_Number 53047-0510 -> 53398-0571; RS Part Number 4476596P -> 542-7292; RS Price/Stock http://uk.rs-online.com/web/p/products/4476596P -> https://uk.rs-online.com/web/p/pcb-headers/5427292; Seeed Part Number (none) -> 53398-0571; now fitted
- R1, R2, R3: Seeed Part Number (none) -> 301010271
- REG1: Seeed Part Number (none) -> AP7361C-33Y5-13
- renumbered J5 to J2, J3 to J4, J4 to J5, U2 to U4, U4 to U5
Connections:
- net +3V3: now also C1.1, C2.1, C3.1, U1.12 (CS), U1.5 (VDDIO), U1.8 (VDD)
- net +BATT: now also U2.15 (BAT)
- net BUTTON_A: now also U2.4 (GPIO4_A3_D3)
- net BUTTON_B: now also U2.5 (GPIO5_A4_D4_SDA)
- net BUZZER_A: now also U2.11 (GPIO9_A10_D10_MOSI)
- net BUZZER_B: now also U2.7 (GPIO43_D6_TX)
- net DRDY: now also U2.10 (GPIO8_A9_D9_MISO)
- net GND: now also C1.2, C2.2, C3.2, U1.1 (SDO/SA0), U1.2 (RES_1), U1.3 (RES_2), U1.6 (GND_1), U1.7 (GND_2), U2.13 (GND)
- net LASER_EN: now also U2.1 (GPIO1_A0_D0)
- net PERIPH_EN: now also U2.6 (GPIO6_A5_D5_SCL)
- net Rx: now also U2.2 (GPIO2_A1_D1)
- net SCL: now also U1.13 (SCL), U2.9 (GPIO7_A8_D8_SCK)
- net SDA: now also U1.14 (SDA), U2.8 (GPIO44_D7_RX)
- net Tx: now also U2.3 (GPIO3_A2_D2)
- net VBUS: now also U2.14 (VBUS)
- no-connect marks 9 -> 18
Other:
- moved on the sheet: C4, C6, R1
