File: hardware/Button/Button.kicad_sch (KiCad schematic)
At the start: 3 parts, among them J1 53048-0310, SW1 SW_Push, SW2 SW_Push

Commit message: More work on the BOM
Parts:
- J0: renamed from J1; Farnell Part Number (none) -> 9732918
- SW1, SW2: Farnell Part Number (none) -> 2396052; Manufacturer_Name (none) -> Alcoswitch - TE Connectivity; Manufacturer_Part_Number (none) -> FSM4JRT
Changed lines of the file:
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@@
     (stroke (width 0) (type default))
   )
-  (label "BUTTON_B" (at 194.31 102.87 180)
+  (label "BUTTON_B" (at 194.31 102.87 180) (fields_autoplaced)
     (effects (font (size 1.27 1.27)) (justify right bottom))
   )
-  (label "BUTTON_B" (at 121.92 106.68 180)
+  (label "BUTTON_B" (at 121.92 106.68 180) (fields_autoplaced)
     (effects (font (size 1.27 1.27)) (justify right bottom))
   )
-  (label "BUTTON_A" (at 194.31 97.79 180)
+  (label "BUTTON_A" (at 194.31 97.79 180) (fields_autoplaced)
     (effects (font (size 1.27 1.27)) (justify right bottom))
   )
-  (label "BUTTON_A" (at 121.92 96.52 180)
+  (label "BUTTON_A" (at 121.92 96.52 180) (fields_autoplaced)
     (effects (font (size 1.27 1.27)) (justify right bottom))
   )
   (symbol (lib_id "Button-rescue:53047-0310-SamacSys") (at 196.85 97.79 0) (unit 1)
     (in_bom yes) (on_board yes) (dnp no)
-    (property "Reference" "J1" (at 212.8012 99.1616 0)
+    (property "Reference" "J0" (at 212.8012 99.1616 0)
       (effects (font (size 1.27 1.27)) (justify left))
     )
@@
       (effects (font (size 1.27 1.27)) (justify left) hide)
     )
+    (property "Farnell Part Number" "9732918 " (at 196.85 97.79 0)
+      (effects (font (size 1.27 1.27)) hide)
+    )
     (pin "3")
     (pin "2")
@@
       (project "Button"
         (path "/99fcb287-88fd-464f-9f69-3e4c0bf057d9"
-          (reference "J1") (unit 1)
+          (reference "J0") (unit 1)
         )
       )
@@
     )
     (property "Datasheet" "~" (at 127 91.44 0)
+      (effects (font (size 1.27 1.27)) hide)
+    )
+    (property "Farnell Part Number" "2396052" (at 127 96.52 0)
+      (effects (font (size 1.27 1.27)) hide)
+    )
+    (property "Manufacturer_Name" "Alcoswitch - TE Connectivity" (at 127 96.52 0)
+      (effects (font (size 1.27 1.27)) hide)
+    )
+    (property "Manufacturer_Part_Number" "FSM4JRT" (at 127 96.52 0)
       (effects (font (size 1.27 1.27)) hide)
     )
@@
       (effects (font (size 1.27 1.27)) hide)
     )
+    (property "Farnell Part Number" "2396052" (at 127 106.68 0)
+      (effects (font (size 1.27 1.27)) hide)
+    )
+    (property "Manufacturer_Name" "Alcoswitch - TE Connectivity" (at 127 106.68 0)
+      (effects (font (size 1.27 1.27)) hide)
+    )
+    (property "Manufacturer_Part_Number" "FSM4JRT" (at 127 106.68 0)
+      (effects (font (size 1.27 1.27)) hide)
+    )

Commit message: update button to kicad8
Parts:
- SW1, SW2: value SW_Push -> FSM4JRT
